File: electrical/internal-psu-v02.kicad_sch (KiCad schematic)
At the start: 15 parts, among them J201 T1 SEC 1, J202 T1 SEC 2, J203 TO AMP J5

Commit message: Update Plan C V0.3 schematics calculations and PDFs
Other:
- note added: "12 VAC auxiliary: reserved for control / speaker protection; AC vs DC module input and current rating TBD."
- note added: "C plan: 20,000 uF per rail. Both bridges and all four reservoir capacitors NOT purchased."
- note added: "Fuse ratings / bridge cooling / inrush / PE chassis bond / speaker protection: design and verify before assembly."
- note added: "INTERNAL LINEAR PSU / V0.3 / PLAN C / SECONDARY-SIDE DRAFT"
- note added: "NEG RAIL / floating 22 VAC secondary"
- note added: "POS RAIL / floating 22 VAC secondary"
- note added: "T1 ordered: 110 VAC primary; 2 x 22 VAC independent + 12 VAC auxiliary. Seller: 200 W; VA / currents TBD."
- note removed: "20,000 uF per rail. GND star is not a substitute for the protective-earth chassis bond."
- note removed: "Bridge pin IDs AC1/AC2/P/N are logical terminals; map to the selected part before assigning any footprint."
- note removed: "F201/F202 ratings, transformer, bridge cooling, primary fuse, inrush control and speaker protection remain TBD."
- note removed: "INTERNAL LINEAR PSU / V0.2 / SECONDARY-SIDE DRAFT"
- note removed: "NEG RAIL / floating 25 VAC secondary"
- note removed: "POS RAIL / floating 25 VAC secondary"
- note removed: "T1 candidate: 300 VA, 2 x 25 VAC INDEPENDENT windings. Primary / soft start shown only in system documentation."
