File: electrical/lm3886-v01.kicad_sch (KiCad schematic)
At the start: 43 parts, among them J1 L RCA, J2 L TEST OUT, J3 R RCA, J4 R TEST OUT, J5 DC +/-35V, U1 LM3886T, U2 LM3886T

Commit message: Plan internal linear power supply and DAC-Z10 RCA power-amp setup
Parts:
- J5: value DC +/-35V -> INTERNAL PSU
Other:
- note added: "J5: internal PSU harness. Bench current-limited supply for first amplifier-only tests."
- note added: "LM3886 / STEREO POWER AMP / EXTERNAL PREAMP / V0.2"
- note added: "Target: 2 x 40 W / 8 ohms. Internal unregulated PSU: approx. +/-33 V loaded; verify actual rails."
- note removed: "LM3886 / SIMPLE STEREO CLASS AB / V0.1"
- note removed: "POWER INPUT: external tracking, current-limited dual supply."
- note removed: "Target: 2 x 40 W into 8 ohms, nominal +/-35 V DC. Draft for review and dummy-load testing."

Commit message: Update Plan C V0.3 schematics calculations and PDFs
Other:
- note added: "LM3886 / STEREO POWER AMP / EXTERNAL PREAMP / V0.3 / PLAN C"
- note added: "Plan C: stereo / 8 ohms / 2 x 22 VAC supply. Output rating TBD by clipping and thermal tests."
- note removed: "LM3886 / STEREO POWER AMP / EXTERNAL PREAMP / V0.2"
- note removed: "Target: 2 x 40 W / 8 ohms. Internal unregulated PSU: approx. +/-33 V loaded; verify actual rails."
