File: electrical/lm3886-v01.kicad_sch (KiCad schematic)
At the start: 43 parts, among them J1 L RCA, J2 L TEST OUT, J3 R RCA, J4 R TEST OUT, J5 INTERNAL PSU, U1 LM3886T, U2 LM3886T

Commit message: rebuild: 原理圖與 PCB 以本機 KiCad 10.0.6 重建，兩板 DRC 0 違規
- 原理圖：ERC 0；verify_electrical 期望值改為實購 100V／0.6W 後通過
- PCB：修正首輪 DRC（C2/R1 保留區重疊、U1 絲印字高與壓字）與回地分組碰觸
  （靜音回流改經 via_mute_ret），DRC 0 違規 0 未連通，verify/analyze/test 通過
- 工具：KiCad 在 Windows 寫出的 CRLF 轉 LF 後才雜湊；雜湊路徑改 as_posix()
- 文件同步；pcb/inspection-v03 與 docs/diagrams 尚未重建

Co-Authored-By: Claude Opus 5.5 (1M context) <noreply@anthropic.com>
Claude-Session: https://claude.ai/code/session_01DerP5HjoiFxZ4hz4f3ygqt
Parts:
- C1, C101: value 2.2u / 63V film -> 2.2u / 100V film
- C103, C104, C3, C4: value 100n / 63V -> 100n / 100V
- C108, C8: value 100u / 63V -> 100u / 100V
- R108, R8: value 22k / 0.25W -> 22k / 0.6W
