File: electrical/control-v01.kicad_sch (KiCad schematic)
At the start: 46 parts, among them J301 T1 12VAC, J302 AMP L OUT -> SPK L+, J303 AMP R OUT -> SPK R+, J304 AMP L JP1 (RUN, VEE), J305 AMP R JP1 (RUN, VEE), J306 TO MAINS K_BYP COIL (BYP_HI, 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, J307 FRONT LED GREEN (A, K), J308 FRONT LED RED (A, K->RLY), J309 GND TO PSU STAR (one point), K301 G2R-1-E 12VDC, K302 G2R-1-E 12VDC, Q301 BC327-40 (PNP, 800 mA), Q302 BC327-40, U301 7812 (TO-220, to chassis), U302 UPC1237 SIP-8, U303 H11D1 (Vceo 300 V), U304 H11D1 (Vceo 300 V), U305 TL431 (2.5 V comparator)

Commit message: pcb: V0.6 控制板 CTRL 70×120 與市電板 MAINS 70×100（DRC 0）；弘宙 102 機箱 3D 配置圖
- 原理圖微調：繼電器全改 Omron G2RL-1-E（KiCad 函式庫有封裝與模型）、輔助電源橋改 1N4007 ×4、光耦 SFH617A-3、補 RLYDRV／ACSENSE 標籤；ERC 0
- 新增 tools/pcb_layout_v06_ctrl.py、build_pcb_v06_ctrl.py（import_std 複製 KiCad 封裝並改焊盤名）、verify_pcb_v06_ctrl.py（含市電／低壓銅箔 ≥6.4 mm 檢查＝7.25）、render_pcb_v06_ctrl.py
- pcb/ctrl-layout-v06、mains-layout-v06 板檔、DRC、JSON、封裝清單、validation-v06-ctrl.json、preview/ctrl-mains-layout-v06.png
- tools/draw_chassis_scene_v06.py（pyvista）→ docs/diagrams/chassis_102_v06_3d.png；.gitignore 補 gltf／STL
- pcb/README、tools/README、HANDOFF、CHANGELOG、docs/00、docs/14 同步

Co-Authored-By: Claude Fable 5.1 <noreply@anthropic.com>
Claude-Session: https://claude.ai/code/session_01TETBHcgmLbP8UasXGwK5UY
Parts:
- removed BR301: DF06M 1A/600V, symbol Project:Bridge
- added D306, D307, D308, D309: 1N4007, symbol Project:D
- K301, K302: value G2R-1-E 12VDC -> G2RL-1-E 12VDC
- U303, U304: value H11D1 (Vceo 300 V) -> SFH617A-3 (Vceo 70 V)
Connections:
- net AC_A: now also D306.2 (A), D308.1 (K)
- net AC_B: now also D307.2 (A), D309.1 (K)
- net GND: now also D308.2 (A), D309.2 (A)
- net RAW: now also D306.1 (K), D307.1 (K)
- net ACSENSE: now reaches D301.1 (K), R306.2
- net RLYDRV: now reaches R303.1, U302.6 (RLY)
Other:
- note added: "C. SPEAKER RELAYS (G2RL-1-E 12VDC, 16 A, 2 x 33 mA), MUTE OPTOS, STATUS LEDS"
- note added: "D306-D309 = full bridge: AC_A/AC_B -> D306/D307 cathodes = RAW; D308/D309 anodes = GND."
- note added: "Opto must stand |VEE| = 36 V when off: SFH617A-3 (70 V, DIP-4) or H11D1 (300 V, DIP-6); NOT PC817 (35 V). LED chain 2 x 1.2 V at ~8 mA from RLY through R309."
- note added: "RAW ~15-17 VDC at ~120 mA (3 x 33 mA G2RL coils + logic). 7812 dissipates ~0.6 W: clip heatsink or bolt to chassis. Ripple 2200u @120 mA ~0.5 Vpp (docs/14 6.5)."
- note added: "Relay DC breaking: G2RL-1-E is rated 30 VDC; a 33.5 V / 8 ohm fault (4.5 A) is a one-shot protective break, accepted 2026-10-01 (docs/14 6.3 asks >=36 VDC)."
- note removed: "C. SPEAKER RELAYS (G2R-1-E 12VDC, 16 A, 2 x 44 mA), MUTE OPTOS, STATUS LEDS"
- note removed: "Opto must stand |VEE| = 36 V when off: H11D1 (300 V) or SFH617A (70 V); NOT PC817 (35 V). LED chain 2 x 1.2 V at ~8 mA from RLY through R309."
- note removed: "RAW ~15-17 VDC at 150 mA (2 x 44 mA coils + bypass coil 44 mA + logic). 7812 dissipates ~1 W: bolt to chassis. Ripple 2200u @150 mA ~0.6 Vpp (docs/14 6.5)."
- note removed: "Relay DC breaking: G2R-1-E is rated 30 VDC; a 33.5 V / 8 ohm fault (4.5 A) is a one-shot protective break, accepted 2026-10-01 (docs/14 6.3 asks >=36 VDC)."
