File: electrical/mains-v01.kicad_sch (KiCad schematic)
At the start: 11 parts, among them J401 FROM IEC + FUSE (L, N), J402 FRONT POWER SWITCH, J403 Z10 12V TRIGGER (tip +, sleev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, J404 FROM CTRL J306 (BYP_HI, GND), J405 TO T1 PRIMARY (L, N), K401 K_TRIG G5LE-1 12VDC (10 A), K402 K_BYP G2R-1-E 12VDC (16 A)

Commit message: pcb: V0.6 控制板 CTRL 70×120 與市電板 MAINS 70×100（DRC 0）；弘宙 102 機箱 3D 配置圖
- 原理圖微調：繼電器全改 Omron G2RL-1-E（KiCad 函式庫有封裝與模型）、輔助電源橋改 1N4007 ×4、光耦 SFH617A-3、補 RLYDRV／ACSENSE 標籤；ERC 0
- 新增 tools/pcb_layout_v06_ctrl.py、build_pcb_v06_ctrl.py（import_std 複製 KiCad 封裝並改焊盤名）、verify_pcb_v06_ctrl.py（含市電／低壓銅箔 ≥6.4 mm 檢查＝7.25）、render_pcb_v06_ctrl.py
- pcb/ctrl-layout-v06、mains-layout-v06 板檔、DRC、JSON、封裝清單、validation-v06-ctrl.json、preview/ctrl-mains-layout-v06.png
- tools/draw_chassis_scene_v06.py（pyvista）→ docs/diagrams/chassis_102_v06_3d.png；.gitignore 補 gltf／STL
- pcb/README、tools/README、HANDOFF、CHANGELOG、docs/00、docs/14 同步

Co-Authored-By: Claude Fable 5.1 <noreply@anthropic.com>
Claude-Session: https://claude.ai/code/session_01TETBHcgmLbP8UasXGwK5UY
Parts:
- K401: value K_TRIG G5LE-1 12VDC (10 A) -> K_TRIG G2RL-1-E 12VDC (16 A)
- K402: value K_BYP G2R-1-E 12VDC (16 A) -> K_BYP G2RL-1-E 12VDC (16 A)
