File: pcb/psu-layout-v03.kicad_pcb (KiCad board)
At the start: 2 copper layers, 160 x 120 mm, 19 parts, among them J201 T1 SEC 1, J202 T1 SEC 2, J203 TO AMP J5

Commit message: pcb: 整流橋定案鎖機殼（方案 A），電源板改 4 位端子並重建，DRC 0
- BridgeTerminal4_P5.08 取代 Bridge_LOGICAL_UNVERIFIED（焊盤編號沿用 AC1/AC2/P/N）
- BR1/BR2 轉 270°，四條 4 mm 進出線加轉折避開相鄰端子
- 電源圖註記、採購總表（§1.1／§2.1，新增 Faston 端子與線材）、HANDOFF、pcb/README、CHANGELOG、README 同步
- 兩板 DRC 0 違規 0 未連通；verify_electrical／power_supply／pcb、analyze、單元測試通過

Co-Authored-By: Claude Fable 5.1 <noreply@anthropic.com>
Claude-Session: https://claude.ai/code/session_01DerP5HjoiFxZ4hz4f3ygqt
Parts:
- BR1, BR2: footprint Bridge_LOGICAL_UNVERIFIED -> BridgeTerminal4_P5.08
- turned BR1 to -90 degrees
- turned BR2 to -90 degrees
Routing:
- net GND: track 362.7 -> 399.9 mm
- net VCC: track 183.5 -> 203.0 mm
- net VEE: track 187.1 -> 204.7 mm
- net POS_AC2: track 35.1 -> 22.7 mm
- net NEG_AC2: track 35.1 -> 22.7 mm
Other:
- board text added: "<- 4 FASTON WIRES"
- board text added: "BR1 KBPC2510 ON CHASSIS"
- board text added: "BR2 KBPC2510 ON CHASSIS"
