File: pcb/mono-layout-v04d.kicad_pcb (KiCad board)
At the start: 2 copper layers, 115 x 90 mm, 26 parts, among them J1 L RCA, J2 L TEST OUT, J5 INTERNAL PSU, U1 LM3886T

Commit message: pcb: 放大板選定 D 為主（C 保留）；D 輸出主幹改頂層，底層鋪銅完整
輸出主幹與 Zobel 接線改 F.Cu，C7→pin1 V+ 改 B.Cu，拿掉 C3.1 多餘 V+ 分支。
DRC 0、鋪銅單一連通區，verify 重綁雜湊。README/CHANGELOG/HANDOFF 記錄決定。

Co-Authored-By: Claude Fable 5.1 <noreply@anthropic.com>
Claude-Session: https://claude.ai/code/session_01DerP5HjoiFxZ4hz4f3ygqt
Routing:
- net VCC: track 94.3 -> 83.0 mm
